File: _saved_rc_car.sch (KiCad schematic (older format))
At the start: 4 parts, among them J1 Conn_01x10_Female, J2 Conn_01x10_Female, U1 L293D, U2 L293D

Commit message: Add files via upload
Parts:
- J1, J2: footprint (none) -> Socket_Strips:Socket_Strip_Angled_1x10_Pitch2.54mm
- U1, U2: footprint (none) -> Pin_Headers:Pin_Header_Straight_2x08_Pitch1.00mm
Changed lines of the file:
@@
 F 0 "U1" H 5650 4650 60  0000 C CNN
 F 1 "L293D" H 5600 2400 60  0000 C CNN
-F 2 "" H 5600 2400 60  0001 C CNN
+F 2 "Pin_Headers:Pin_Header_Straight_2x08_Pitch1.00mm" H 5600 2400 60  0001 C CNN
 F 3 "" H 5600 2400 60  0001 C CNN
 	1    5650 3550
@@
 F 0 "U2" H 8550 4550 60  0000 C CNN
 F 1 "L293D" H 8500 2300 60  0000 C CNN
-F 2 "" H 8500 2300 60  0001 C CNN
+F 2 "Pin_Headers:Pin_Header_Straight_2x08_Pitch1.00mm" H 8500 2300 60  0001 C CNN
 F 3 "" H 8500 2300 60  0001 C CNN
 	1    8550 3450
@@
 F 0 "J1" H 2850 3950 50  0000 C CNN
 F 1 "Conn_01x10_Female" H 2850 2850 50  0000 C CNN
-F 2 "" H 2850 3450 50  0001 C CNN
+F 2 "Socket_Strips:Socket_Strip_Angled_1x10_Pitch2.54mm" H 2850 3450 50  0001 C CNN
 F 3 "" H 2850 3450 50  0001 C CNN
 	1    2850 3450
@@
 F 0 "J2" H 10400 3750 50  0000 C CNN
 F 1 "Conn_01x10_Female" H 10400 2650 50  0000 C CNN
-F 2 "" H 10400 3250 50  0001 C CNN
+F 2 "Socket_Strips:Socket_Strip_Angled_1x10_Pitch2.54mm" H 10400 3250 50  0001 C CNN
 F 3 "" H 10400 3250 50  0001 C CNN
 	1    10400 3250
