File: rc_car.sch (KiCad schematic (older format))
At the start: 4 parts

Commit message: Add files via upload
Parts:
- J1, J2: renamed from J?; footprint (none) -> Socket_Strips:Socket_Strip_Angled_1x01_Pitch2.00mm
- U1, U2: renamed from U?; footprint (none) -> Pin_Headers:Pin_Header_Angled_2x16_Pitch1.00mm
Changed lines of the file:
@@
 $EndDescr
 $Comp
-L L293D U?
+L L293D U1
 U 1 1 5AC29786
 P 5650 3550
-F 0 "U?" H 5650 4650 60  0000 C CNN
+F 0 "U1" H 5650 4650 60  0000 C CNN
 F 1 "L293D" H 5600 2400 60  0000 C CNN
-F 2 "" H 5600 2400 60  0001 C CNN
+F 2 "Pin_Headers:Pin_Header_Angled_2x16_Pitch1.00mm" H 5600 2400 60  0001 C CNN
 F 3 "" H 5600 2400 60  0001 C CNN
 	1    5650 3550
@@
 $EndComp
 $Comp
-L L293D U?
+L L293D U2
 U 1 1 5AC2983D
 P 8550 3450
-F 0 "U?" H 8550 4550 60  0000 C CNN
+F 0 "U2" H 8550 4550 60  0000 C CNN
 F 1 "L293D" H 8500 2300 60  0000 C CNN
-F 2 "" H 8500 2300 60  0001 C CNN
+F 2 "Pin_Headers:Pin_Header_Angled_2x16_Pitch1.00mm" H 8500 2300 60  0001 C CNN
 F 3 "" H 8500 2300 60  0001 C CNN
 	1    8550 3450
@@
 $EndComp
 $Comp
-L GND #PWR?
+L GND #PWR01
 U 1 1 5AC29899
 P 6800 1500
-F 0 "#PWR?" H 6800 1250 50  0001 C CNN
+F 0 "#PWR01" H 6800 1250 50  0001 C CNN
 F 1 "GND" H 6800 1350 50  0000 C CNN
 F 2 "" H 6800 1500 50  0001 C CNN
@@
 $EndComp
 $Comp
-L Conn_01x10_Female J?
+L Conn_01x10_Female J1
 U 1 1 5AC298B1
 P 2850 3450
-F 0 "J?" H 2850 3950 50  0000 C CNN
+F 0 "J1" H 2850 3950 50  0000 C CNN
 F 1 "Conn_01x10_Female" H 2850 2850 50  0000 C CNN
-F 2 "" H 2850 3450 50  0001 C CNN
+F 2 "Socket_Strips:Socket_Strip_Angled_1x01_Pitch2.00mm" H 2850 3450 50  0001 C CNN
 F 3 "" H 2850 3450 50  0001 C CNN
 	1    2850 3450
@@
 $EndComp
 $Comp
-L Conn_01x10_Female J?
+L Conn_01x10_Female J2
 U 1 1 5AC2991C
 P 10400 3250
-F 0 "J?" H 10400 3750 50  0000 C CNN
+F 0 "J2" H 10400 3750 50  0000 C CNN
 F 1 "Conn_01x10_Female" H 10400 2650 50  0000 C CNN
-F 2 "" H 10400 3250 50  0001 C CNN
+F 2 "Socket_Strips:Socket_Strip_Angled_1x01_Pitch2.00mm" H 10400 3250 50  0001 C CNN
 F 3 "" H 10400 3250 50  0001 C CNN
 	1    10400 3250
@@
 $EndComp
 $Comp
-L VCC #PWR?
+L VCC #PWR02
 U 1 1 5AC29BE5
 P 7350 1650
-F 0 "#PWR?" H 7350 1500 50  0001 C CNN
+F 0 "#PWR02" H 7350 1500 50  0001 C CNN
 F 1 "VCC" H 7350 1800 50  0000 C CNN
 F 2 "" H 7350 1650 50  0001 C CNN
